File: pcb-design/pcb-design.kicad_sch (KiCad schematic)
At the start: 24 parts, among them SW1 SW_Push, U1 ATmega32U4-A, Y1 16MHz

Commit message: started PCB placement
Parts:
- C7: value 0.1uF -> 10uF
Changed lines of the file:
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@@
       (effects (font (size 1.27 1.27)) (justify left))
     )
-    (property "Value" "0.1uF" (id 1) (at 209.55 106.6862 0)
+    (property "Value" "10uF" (id 1) (at 209.55 106.6862 0)
       (effects (font (size 1.27 1.27)) (justify left))
     )
@@
     )
     (path "/bc415191-2264-432a-91a2-21b0cf8e7e17"
-      (reference "C7") (unit 1) (value "0.1uF") (footprint "Capacitor_SMD:C_0805_2012Metric")
+      (reference "C7") (unit 1) (value "10uF") (footprint "Capacitor_SMD:C_0805_2012Metric")
     )
     (path "/b68d8a82-0ba5-463e-b05f-7ad6a1e19336"
